File: KiCAD/EMDR-Device.kicad_pcb (KiCad board)
At the start: 2 copper layers, 65 x 32.5 mm, 0 parts

Commit message: schematic
Parts:
- added C1: 0.1uF, Capacitor_SMD:C_0603_1608Metric, B.Cu at (129.9, 121.4)
- added C10: 0.1uF, Capacitor_SMD:C_0603_1608Metric, B.Cu at (133.8, 99.7)
- added C11: 10uF, Capacitor_SMD:C_0603_1608Metric, B.Cu at (129.9, 134.0)
- added C13: 0.1uF, Capacitor_SMD:C_0603_1608Metric, B.Cu at (133.8, 106.7)
- added C14: 0.1uF, Capacitor_SMD:C_0603_1608Metric, B.Cu at (133.8, 109.2)
- added C15: 0.1uF, Capacitor_SMD:C_0603_1608Metric, B.Cu at (133.8, 111.7)
- added C16: 0.1uF, Capacitor_SMD:C_0603_1608Metric, B.Cu at (148.0, 121.7)
- added C2: 10uF, Capacitor_SMD:C_0603_1608Metric, B.Cu at (129.9, 123.9)
- added C3: 1uF, Capacitor_SMD:C_0603_1608Metric, B.Cu at (129.9, 126.5)
- added C4: 1uF, Capacitor_SMD:C_0603_1608Metric, B.Cu at (153.0, 104.4)
- added C5: 0.1uF, Capacitor_SMD:C_0603_1608Metric, B.Cu at (129.9, 129.0)
- added C6: 1uF, Capacitor_SMD:C_0603_1608Metric, B.Cu at (129.9, 131.5)
- added C7: 1uF, Capacitor_SMD:C_0603_1608Metric, B.Cu at (153.0, 106.9)
- added C8: 10uF, Capacitor_SMD:C_0603_1608Metric, B.Cu at (153.0, 121.4)
- added C9: 10uF, Capacitor_SMD:C_0603_1608Metric, B.Cu at (153.0, 123.9)
- added D1: LED, LED_SMD:LED_0603_1608Metric, B.Cu at (140.9, 131.1)
- added D2: SS14, Diode_SMD:D_SMA, B.Cu at (147.0, 132.1)
- added H1: MountingHole, MountingHole:MountingHole_3.2mm_M3_DIN965_Pad, F.Cu at (205.4, 115.1)
- added H2: MountingHole, MountingHole:MountingHole_3.2mm_M3_DIN965_Pad, F.Cu at (205.4, 122.3)
- added H3: MountingHole, MountingHole:MountingHole_3.2mm_M3_DIN965_Pad, F.Cu at (205.4, 129.4)
- added H4: MountingHole, MountingHole:MountingHole_3.2mm_M3_DIN965_Pad, F.Cu at (205.4, 136.6)
- added J1: USB_C_Receptacle_USB2.0_14P, Connector_USB:USB_C_Receptacle_HCTL_HC-TYPE-C-16P-01A, B.Cu at (162.8, 121.6)
- added J2: Conn_01x02_Socket, Connector_JST:JST_PH_S2B-PH-K_1x02_P2.00mm_Horizontal, B.Cu at (172.2, 123.7)
- added Q1: AO3401A, Package_TO_SOT_SMD:SOT-23, B.Cu at (140.6, 127.0)
- added R10: 200k, Resistor_SMD:R_0603_1608Metric, B.Cu at (153.0, 134.0)
- added R11: 200k, Resistor_SMD:R_0603_1608Metric, B.Cu at (153.0, 136.5)
- added R12: 10k, Resistor_SMD:R_0603_1608Metric, B.Cu at (153.0, 114.4)
- added R13: 10k, Resistor_SMD:R_0603_1608Metric, B.Cu at (153.0, 116.9)
- added R18: 10k, Resistor_SMD:R_0603_1608Metric, B.Cu at (133.8, 102.2)
- added R5: 5.1k, Resistor_SMD:R_0603_1608Metric, B.Cu at (153.0, 109.4)
- added R6: 5.1k, Resistor_SMD:R_0603_1608Metric, B.Cu at (153.0, 111.9)
- added R7: 1k, Resistor_SMD:R_0603_1608Metric, B.Cu at (153.0, 126.5)
- added R8: 2k, Resistor_SMD:R_0603_1608Metric, B.Cu at (153.0, 129.0)
- added R9: 100k, Resistor_SMD:R_0603_1608Metric, B.Cu at (153.0, 131.5)
- added TP1: TestPoint, Connector_Pin:Pin_D1.0mm_L10.0mm, B.Cu at (133.9, 122.2)
- added TP2: TestPoint, Connector_Pin:Pin_D1.0mm_L10.0mm, B.Cu at (133.9, 126.2)
- added TP3: TestPoint, Connector_Pin:Pin_D1.0mm_L10.0mm, B.Cu at (133.9, 130.3)
- added TP4: TestPoint, Connector_Pin:Pin_D1.0mm_L10.0mm, B.Cu at (133.9, 134.3)
- added U1: ER_OLEDM0.91_1x-I2C, Display:ER_OLEDM0.91_1x-I2C, F.Cu at (206.0, 72.3)
- added U2: ESP32-C6-MINI-1, RF_Module:ESP32-C6-MINI-1, B.Cu at (179.8, 102.0)
- added U3: DRV2605LDGS, Package_SO:TSSOP-10_3x3mm_P0.5mm, B.Cu at (124.2, 122.5)
- added U4: DRV2605LDGS, Package_SO:TSSOP-10_3x3mm_P0.5mm, B.Cu at (124.2, 127.0)
- added U5: MCP73831-2-OT, Package_TO_SOT_SMD:SOT-23-5, B.Cu at (140.5, 122.6)
- added U6: XC6206PxxxMR, Package_TO_SOT_SMD:SOT-23-3, B.Cu at (148.4, 115.5)
- added U7: TCA9546APW, Package_SO:TSSOP-16_4.4x5mm_P0.65mm, B.Cu at (131.0, 95.1)
- added U8: LSM6DS3, Package_LGA:LGA-14_3x2.5mm_P0.5mm_LayoutBorder3x4y, B.Cu at (129.1, 107.5)
Routing:
- removed copper zone on B.Cu, net GND
- removed copper zone on F.Cu, net GND

Commit message: preliminary pcb
Parts:
- added C12: 1uF, Capacitor_SMD:C_0603_1608Metric, B.Cu at (234.4, 112.5)
- added C17: 15pF, Capacitor_SMD:C_0603_1608Metric, B.Cu at (234.4, 115.0)
- added R14: 5.1k, Resistor_SMD:R_0603_1608Metric, B.Cu at (234.4, 117.5)
- added R15: 10k, Resistor_SMD:R_0603_1608Metric, B.Cu at (234.4, 120.0)
- added R16: 10k, Resistor_SMD:R_0603_1608Metric, B.Cu at (234.4, 122.5)
- added SW1: Switch, Button_Switch_SMD:Panasonic_EVQPUJ_EVQPUA, B.Cu at (152.1, 85.8)
- added SW2: Switch, Button_Switch_SMD:Panasonic_EVQPUJ_EVQPUA, B.Cu at (142.3, 85.8)
- moved H1 86.0 mm to (123.5, 89.0)
- moved H3 83.9 mm to (123.5, 111.5)
- moved U1 79.2 mm to (133.5, 104.1), turned to 90 degrees
- moved U8 59.4 mm to (180.9, 136.6), turned to 0 degrees
- moved J2 57.0 mm to (122.5, 95.9), turned to -90 degrees
- moved H2 42.8 mm to (178.5, 89.0)
- moved C10 41.1 mm to (153.7, 135.7)
- moved C14 41.1 mm to (153.7, 145.2)
- moved Q1 41.1 mm to (160.6, 163.0)
- moved TP1 41.1 mm to (153.8, 158.2)
- moved U5 41.1 mm to (160.4, 158.6)
- moved C13 41.1 mm to (153.7, 142.7)
- moved C15 41.1 mm to (153.7, 147.7)
- moved D1 41.1 mm to (160.8, 167.1)
- moved R18 41.1 mm to (153.7, 138.2)
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Connections:
- C1 pad 1: +5V -> V_SYS
- C11 pad 1: +5V -> V_SYS
- C2 pad 1: +5V -> V_SYS
- C5 pad 1: +5V -> V_SYS
- U2 pad 19: unconnected-(U2-IO14-Pad19) -> in/trig_1
- U2 pad 20: unconnected-(U2-IO15-Pad20) -> in/trig_2
- U2 pad 22: unconnected-(U2-IO8-Pad22) -> Net-(U2-IO8)
- U2 pad 23: unconnected-(U2-IO9-Pad23) -> BOOT
- U2 pad 5: unconnected-(U2-IO2-Pad5) -> INT1
- U2 pad 6: unconnected-(U2-IO3-Pad6) -> INT2
- U3 pad 10: +5V -> V_SYS
- U3 pad 5: +5V -> V_SYS
- U3 pad 6: +5V -> V_SYS
- U4 pad 10: +5V -> V_SYS
- U4 pad 5: +5V -> V_SYS
- U4 pad 6: +5V -> V_SYS
- U8 pad 4: unconnected-(U8-INT1-Pad4) -> INT1
- U8 pad 9: unconnected-(U8-INT2-Pad9) -> INT2
Routing:
- net D_N: track 0.00 -> 2.59 mm
- net D_P: track 0.00 -> 2.59 mm

Commit message: full pcb
Parts:
- moved R16 96.5 mm to (145.1, 86.0), turned to -90 degrees
- moved C17 92.4 mm to (146.7, 85.9), turned to 90 degrees
- moved R15 84.7 mm to (156.8, 85.9), turned to -90 degrees
- moved R11 84.6 mm to (125.9, 92.9), turned to 0 degrees
- moved Q1 81.2 mm to (129.3, 88.1), turned to 0 degrees
- moved R10 80.8 mm to (129.5, 92.5), turned to 0 degrees
- moved R8 80.7 mm to (122.0, 93.0)
- moved C12 80.4 mm to (158.4, 85.9), turned to 90 degrees
- moved R9 78.4 mm to (132.0, 91.2), turned to 90 degrees
- moved D1 77.9 mm to (123.1, 98.9), turned to 90 degrees
- moved D2 76.2 mm to (134.6, 89.7), turned to -90 degrees
- moved C9 73.9 mm to (129.6, 90.7)
- moved U5 72.8 mm to (124.0, 95.5)
- moved R7 72.5 mm to (124.7, 98.9), turned to 90 degrees
- moved C8 69.1 mm to (129.6, 94.2)
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Routing:
- net V_SYS: track 0.00 -> 84.0 mm, vias 0 -> 4
- net +5V: track 0.00 -> 82.1 mm, vias 0 -> 5
- net i2c_scl: track 0.00 -> 70.2 mm, vias 0 -> 1
- net i2c_sda: track 0.00 -> 69.8 mm, vias 0 -> 1
- net BAT: track 0.00 -> 61.5 mm, vias 0 -> 2
- net EN: track 0.00 -> 46.7 mm, vias 0 -> 2
- net BOOT: track 0.00 -> 41.7 mm, vias 0 -> 2
- net INT1: track 0.00 -> 40.4 mm, vias 0 -> 2
- net GND: track 0.00 -> 37.6 mm, vias 0 -> 16
- net INT2: track 0.00 -> 32.7 mm, vias 0 -> 2
- net +3V3: track 0.00 -> 30.5 mm, vias 0 -> 12
- net Net-(U4-OUT-): track 0.00 -> 29.0 mm
- net Net-(U4-OUT+): track 0.00 -> 27.4 mm
- net BAT_RAW_P: track 0.00 -> 25.8 mm
- net Net-(U3-OUT-): track 0.00 -> 24.9 mm
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- added copper zone on In2.Cu, net +3V3
- added copper zone on B.Cu, net GND
- added copper zone on F.Cu, net GND
- added copper zone on In1.Cu, net GND
Other:
- copper layers 2 -> 4
- board text added: "Motor 1 +"
- board text added: "Motor 1 -"
- board text added: "Motor 2 +"
- board text added: "Motor 2 -"
